File: CUTIE-ZEST.kicad_sch (KiCad schematic)
At the start: 17 parts, among them U1 TCAN334, U2 MCP98243, U3 ADP7158ACPZ-3.3-R7

Commit message: bom for assembly
Parts:
- C1, C2: Manufacturer (none) -> KEMET; Manufacturer Product Number (none) -> C0402C104K4RACTU
- C3, C4: Manufacturer (none) -> Taiyo Yuden; Manufacturer Product Number (none) -> LMK107BBJ106MALT
- C5, C6, C7: Manufacturer (none) -> KEMET; Manufacturer Product Number (none) -> C0603C105K4RACTU
- D3: Manufacturer (none) -> Lite-On Inc.; Manufacturer Product Number (none) -> LTST-C171KGKT
- R9: Manufacturer (none) -> Panasonic Electronic Components; Manufacturer Product Number (none) -> ERA-2AEB222X
- TP1, TP2, TP3, TP4, TP5: now left out of the parts list
- U2: Manufacturer (none) -> Microchip Technology; Manufacturer Product Number (none) -> MCP98243T-BE/MC
- U3: Manufacturer (none) -> Analog Devices Inc.; Manufacturer Product Number (none) -> ADP7158ACPZ-3.3-R7
