File: CUTIE-ZEST.kicad_pcb (KiCad board)
At the start: 4 copper layers, 78.5 x 78.5 mm, 64 parts, among them J1 TC2030, J2 U.FL, J3 U.FL, P1 ERM8-025-01-L-D-RA-K-TR, U1 TCAN334, U2 MCP98243, U3 ADP7158ACPZ-3.3-R7, U4 STM32G474CEUx, U5 AS179-92LF, U6 SX1262IMLTRT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

Commit message: update for prod
Parts:
- added G***: LOGO, LOGO, B.Cu at (150.0, 130.0)
