File: sch/backplane.kicad_sch (KiCad schematic)
At the start: 3 parts, among them P1 ERM8-025-01-L-D-RA-K-TR

Commit message: bom for assembly
Parts:
- D2: Manufacturer (none) -> Lite-On Inc.; Manufacturer Product Number (none) -> LTST-C171KRKT
- P1: Manufacturer (none) -> Samtec Inc.; Manufacturer Product Number (none) -> ERM8-025-01-L-D-RA-K-TR
- R7: Manufacturer (none) -> Panasonic Electronic Components; Manufacturer Product Number (none) -> ERA-2AEB222X
Changed lines of the file:
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@@
 (kicad_sch
-	(version 20260101)
+	(version 20260306)
 	(generator "eeschema")
-	(generator_version "9.99")
+	(generator_version "10.0")
 	(paper "A4")
 	(junction
@@
 			)
 		)
-		(property "Description" ""
+		(property "Description" "CONN HDR 50POS R/A SMD GOLD"
+			(at 144.78 93.98 0)
+			(hide yes)
+			(show_name no)
+			(do_not_autoplace no)
+			(effects
+				(font
+					(size 1.27 1.27)
+				)
+			)
+		)
+		(property "Manufacturer" "Samtec Inc."
+			(at 144.78 93.98 0)
+			(hide yes)
+			(show_name no)
+			(do_not_autoplace no)
+			(effects
+				(font
+					(size 1.27 1.27)
+				)
+			)
+		)
+		(property "Manufacturer Product Number" "ERM8-025-01-L-D-RA-K-TR"
 			(at 144.78 93.98 0)
 			(hide yes)
@@
 			)
 		)
-		(property "Description" "Resistor, US symbol"
+		(property "Description" "RES SMD 2.2K OHM 0.1% 1/16W 0402"
+			(at 111.76 133.35 0)
+			(hide yes)
+			(show_name no)
+			(do_not_autoplace no)
+			(effects
+				(font
+					(size 1.27 1.27)
+				)
+			)
+		)
+		(property "Manufacturer" "Panasonic Electronic Components"
+			(at 111.76 133.35 0)
+			(hide yes)
+			(show_name no)
+			(do_not_autoplace no)
+			(effects
+				(font
+					(size 1.27 1.27)
+				)
+			)
+		)
+		(property "Manufacturer Product Number" "ERA-2AEB222X"
 			(at 111.76 133.35 0)
 			(hide yes)
@@
 			)
 		)
-		(property "Description" "Light emitting diode"
+		(property "Description" "LED RED CLEAR SMD"
 			(at 111.76 123.19 0)
 			(hide yes)
@@
 			(hide yes)
 			(show_name no)
+			(do_not_autoplace no)
+			(effects
+				(font
+					(size 1.27 1.27)
+				)
+			)
+		)
+		(property "Manufacturer" "Lite-On Inc."
+			(at 111.76 123.19 90)
+			(hide yes)
+			(show_name no)
+			(do_not_autoplace no)
+			(effects
+				(font
+					(size 1.27 1.27)
+				)
+			)
+		)
+		(property "Manufacturer Product Number" "LTST-C171KRKT"
+			(at 111.76 123.19 90)
+			(hide yes)
+			(show_name no)
