File: sch/rf.kicad_sch (KiCad schematic)
At the start: 27 parts, among them J2 U.FL, J3 U.FL, U5 AS179-92LF, U6 SX1262IMLTRT, U7 SN74LVC1G14DBV, U8 NEO-M8M, Y1 ECS-TXO-2520MV

Commit message: bom for assembly
Parts:
- C13: Manufacturer (none) -> KEMET; Manufacturer Product Number (none) -> C0402C103K3REC7411
- C14, C18, C21, C22, C23, C26, C27: Manufacturer (none) -> KEMET; Manufacturer Product Number (none) -> C0402C104K4RACTU
- C15, C16, C17, C19, C24, C25: Manufacturer (none) -> Murata Electronics; Manufacturer Product Number (none) -> GRM1555C1H470JA01D
- C20: Manufacturer (none) -> TDK; Manufacturer Product Number (none) -> C1005X5R1E474K050BB
- FB1: Manufacturer (none) -> Murata Electronics; Manufacturer Product Number (none) -> BLM21PG300SN1D
- FL1: Manufacturer (none) -> Johanson Technology Inc.; Manufacturer Product Number (none) -> 0900FM15K0039001E
- J2, J3: Manufacturer (none) -> Hirose Electric Co Ltd; Manufacturer Product Number (none) -> U.FL-R-SMT-1(10)
- L1, L2: Manufacturer (none) -> Murata Electronics; Manufacturer Product Number (none) -> LQW15AN47NJ00D
- R1: Manufacturer (none) -> Vishay Dale; Manufacturer Product Number (none) -> CRCW040210R0FKED
- U5: Manufacturer (none) -> Skyworks Solutions Inc.; Manufacturer Product Number (none) -> AS179-92LF
- U6: Manufacturer (none) -> Semtech Corporation; Manufacturer Product Number (none) -> SX1262IMLTRT
- U7: Manufacturer (none) -> Texas Instruments; Manufacturer Product Number (none) -> SN74LVC1G14DBVT
- U8: Manufacturer (none) -> u-blox; Manufacturer Product Number (none) -> NEO-M8M-0
- Y1: Manufacturer (none) -> ECS Inc.; Manufacturer Product Number (none) -> ECS-TXO-2520MV-100-AN-TR
