File: sch/stm32.kicad_sch (KiCad schematic)
At the start: 15 parts, among them J1 TC2030, U4 STM32G474CEUx

Commit message: bom for assembly
Parts:
- C10, C11, C12, C9: Manufacturer (none) -> KEMET; Manufacturer Product Number (none) -> C0402C104K4RACTU
- C8: Manufacturer (none) -> Murata Electronics; Manufacturer Product Number (none) -> GRM188R61E475KE11D
- D1: Manufacturer (none) -> Lite-On Inc.; Manufacturer Product Number (none) -> LTST-C170TBKT
- R2, R3, R4, R5, R6: Manufacturer (none) -> YAGEO; Manufacturer Product Number (none) -> RC0402JR-074K7L
- R8: Manufacturer (none) -> YAGEO; Manufacturer Product Number (none) -> RC0402FR-07330RL
- TP6: now left out of the parts list
- U4: Manufacturer (none) -> STMicroelectronics; Manufacturer Product Number (none) -> STM32G474CEU6

Commit message: push for fab
Parts:
- U4: value STM32G474CEUx -> STM32G473CEU6; Manufacturer Product Number STM32G474CEU6 -> STM32G473CEU6
Changed lines of the file:
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@@
 			)
 		)
-		(property "Value" "STM32G474CEUx"
+		(property "Value" "STM32G473CEU6"
 			(at 134.62 50.8 0)
 			(show_name no)
@@
 			)
 		)
-		(property "Manufacturer Product Number" "STM32G474CEU6"
+		(property "Manufacturer Product Number" "STM32G473CEU6"
 			(at 134.62 91.44 0)
 			(hide yes)
